File: Infrarooi LED Alarm met 555 timer IC.sch (KiCad schematic (older format))
At the start: 11 parts, among them U1 LM358N, U2 NE555

Commit message: CAp toevoeging
Parts:
- D1: symbol LED -> LED-RESCUE-Infrarooi_LED_Alarm_met_555_timer_IC
- RV1: symbol POT -> POT-RESCUE-Infrarooi_LED_Alarm_met_555_timer_IC
Other:
- moved on the sheet: C1, D1, R1, R2, R3, R4, R5, RV1, SP1, U1A, U2
